File: PMIC_module.kicad_pcb (KiCad board)
At the start: 2 copper layers, 14 parts, among them J1 Conn_01x04_Pin, J2 Conn_01x02_Pin, J3 Conn_01x02_Pin, J4 Conn_01x02_Pin, J5 Conn_01x04_Pin, U1 MAX17048G+T10, U2 MCP73832-2-OT

Commit message: PMIC Gbr
Parts:
- removed J5: Conn_01x04_Pin, Connector_JST:JST_PH_B4B-PH-SM4-TB_1x04-1MP_P2.00mm_Vertical
- removed TP1: TestPoint_Small, Connector_Wire:SolderWire-0.1sqmm_1x01_D0.4mm_OD1mm
- added JP1: SolderJumper_3_Open, Jumper:SolderJumper-3_P1.3mm_Open_Pad1.0x1.5mm, F.Cu at (91.2, 83.8)
- added JP2: SolderJumper_2_Open, Jumper:SolderJumper-2_P1.3mm_Open_Pad1.0x1.5mm, F.Cu at (81.3, 83.8)
- added R3: 2.2K, Resistor_SMD:R_0603_1608Metric_Pad0.98x0.95mm_HandSolder, F.Cu at (90.4, 86.6)
- added R4: 2.2K, Resistor_SMD:R_0603_1608Metric_Pad0.98x0.95mm_HandSolder, F.Cu at (94.3, 86.6)
- added R5: 10K, Resistor_SMD:R_0603_1608Metric_Pad0.98x0.95mm_HandSolder, F.Cu at (85.8, 83.8)
- J2: value Conn_01x02_Pin -> Conn_01x04_Pin; footprint Connector_JST:JST_PH_S2B-PH-SM4-TB_1x02-1MP_P2.00mm_Horizontal -> Castellated_PinHeaders_1x04:Castellated_PinHeader_1x04_P2.54mm
- J3: value Conn_01x02_Pin -> Conn_01x04_Pin; footprint Connector_Wire:SolderWire-0.1sqmm_1x02_P3.6mm_D0.4mm_OD1mm -> Connector_JST:JST_PH_B4B-PH-SM4-TB_1x04-1MP_P2.00mm_Vertical
- J4: footprint Connector_Wire:SolderWire-0.1sqmm_1x02_P3.6mm_D0.4mm_OD1mm -> Connector_JST:JST_PH_S2B-PH-SM4-TB_1x02-1MP_P2.00mm_Horizontal
- R1: value 10K -> 2K
- R2: value 2K -> 10K
- moved J1 110.0 mm to (102.0, 94.4), turned to 180 degrees
- moved U1 82.0 mm to (90.7, 90.1), turned to 0 degrees
- moved C1 79.4 mm to (91.4, 94.0)
- moved J4 75.5 mm to (94.0, 101.6), turned to 0 degrees
- moved U2 67.5 mm to (85.0, 89.7)
- moved J3 62.7 mm to (82.3, 102.1)
- moved C2 58.7 mm to (81.3, 94.0), turned to 180 degrees
- moved C3 57.0 mm to (86.4, 94.0), turned to 180 degrees
- moved R1 47.0 mm to (85.9, 86.4)
- moved J2 46.8 mm to (73.8, 86.4), turned to 0 degrees
- moved R2 43.7 mm to (81.3, 86.4)
- moved D1 33.1 mm to (81.3, 89.7), turned to -90 degrees
Connections:
- C1 pad 1: BAT -> +BATT
- C2 pad 1: GND -> +BATT
- C2 pad 2: BAT -> GND
- C3 pad 1: VCC -> GND
- C3 pad 2: GND -> +BATT
- J1 pad : (no net) -> GND
- J1 pad 1: GND -> SDA_PMIC
- J1 pad 2: ALERT -> SCL_PMIC
- J1 pad 3: SCL_PMIC -> +BATT
- J1 pad 4: SDA_PMIC -> GND
- J2 pad 2: BAT -> ALERT
- J4 pad 1: SCL_PMIC -> GND
- J4 pad 2: SDA_PMIC -> +BATT
- R1 pad 1: Net-(D1-K) -> GND
- R1 pad 2: GND -> Net-(U2-PROG)
- R2 pad 1: GND -> Net-(D1-K)
- R2 pad 2: Net-(U2-PROG) -> GND
- U1 pad 2: BAT -> +BATT
- U1 pad 3: BAT -> +BATT
- U2 pad 3: BAT -> +BATT
- U2 pad 4: VCC -> +BATT
Routing:
- net GND: track 0.00 -> 93.3 mm, vias 0 -> 5
- net SDA_PMIC: track 0.00 -> 62.0 mm, vias 0 -> 1
- net +BATT: track 0.00 -> 61.8 mm, vias 0 -> 2
- net SCL_PMIC: track 0.00 -> 56.2 mm, vias 0 -> 1
- net ALERT: track 0.00 -> 25.3 mm
- net Net-(D1-A): track 0.00 -> 3.27 mm
- net Net-(JP1-A): track 0.00 -> 3.07 mm
- net Net-(JP2-B): track 0.00 -> 2.98 mm
- net Net-(U2-PROG): track 0.00 -> 2.89 mm
- net Net-(JP1-B): track 0.00 -> 2.89 mm
- net Net-(D1-K): track 0.00 -> 2.83 mm
Other:
- board outline added: 28.1 x 30.4 mm
