File: PMIC_module.kicad_sch (KiCad schematic)
At the start: 13 parts, among them J1 Conn_01x04_Pin, J2 Conn_01x02_Pin, J3 Conn_01x02_Pin, J4 Conn_01x02_Pin, J5 Conn_01x04_Pin, U1 MAX17048G+T10, U2 MCP73832-2-OT

Commit message: PMIC Gbr
Parts:
- removed J3, J4: Conn_01x02_Pin, Connector_Wire:SolderWire-0.1sqmm_1x02_P3.6mm_D0.4mm_OD1mm, symbol Connector:Conn_01x02_Pin
- added J1: Conn_01x04_Pin, Castellated_PinHeaders_1x04:Castellated_PinHeader_1x04_P2.54mm, symbol Connector:Conn_01x04_Pin
- added JP1: SolderJumper_3_Open, Jumper:SolderJumper-3_P1.3mm_Open_Pad1.0x1.5mm, symbol Jumper:SolderJumper_3_Open
- added JP2: SolderJumper_2_Open, Jumper:SolderJumper-2_P1.3mm_Open_Pad1.0x1.5mm, symbol Jumper:SolderJumper_2_Open
- added R3, R4: 2.2K, Resistor_SMD:R_0603_1608Metric_Pad0.98x0.95mm_HandSolder, symbol Device:R
- added R5: 10K, Resistor_SMD:R_0603_1608Metric_Pad0.98x0.95mm_HandSolder, symbol Device:R
- renumbered C3 to C2, C2 to C3, J1 to J2, J5 to J3, J2 to J4, R2 to R1, R1 to R2
Connections:
- net ALERT: now also JP2.1 (A)
- net GND: now also J1.4 (Pin_4)
- net SCL_PMIC: now also J3.4 (Pin_4), J1.2 (Pin_2), R4.1; no longer J3.3 (Pin_3)
- net SDA_PMIC: now also J3.3 (Pin_3), J1.1 (Pin_1), R3.1; no longer J3.4 (Pin_4)
- net BAT renamed +BATT
- net +BATT: now also C2.1, U2.4 (V_{DD}), J1.3 (Pin_3), JP1.2 (C), R5.2
- removed net VCC: C2.1, J3.2 (Pin_2), U2.4 (V_{DD})
- new net: JP1.1 (A), R4.2
- new net: JP1.3 (B), R3.2
- new net: JP2.2 (B), R5.1
- no-connect marks 0 -> 1
Other:
- sheet Connectors_BAT renamed Qwiic
- added sheet Pull-up registers (Pull-ups.kicad_sch)
- note added: "Charging circuit"
- note added: "Connectors"
- note added: "Pull-ups"
- note added: "Voltage sensing"
- company: (none) -> WBL
- title: (none) -> PMIC_Minder
- moved on the sheet: J2, J3, J4
